File: pcb_layouts/ProgramCount/ProgramCount.kicad_pcb (KiCad board)
At the start: 2 copper layers, 135 x 120 mm, 6 parts, among them J1 Conn_02x20_Odd_Even, J2 Conn_02x20_Odd_Even

Commit message: pcbs
Parts:
- added C10: 22uf, Capacitor_THT:CP_Radial_D4.0mm_P2.00mm, F.Cu at (248.0, 92.9)
- added C11: 22uf, Capacitor_THT:CP_Radial_D4.0mm_P2.00mm, F.Cu at (223.2, 118.3)
- added C5: 22uf, Capacitor_THT:CP_Radial_D4.0mm_P2.00mm, F.Cu at (248.0, 87.3)
- added C6: 22uf, Capacitor_THT:CP_Radial_D4.0mm_P2.00mm, F.Cu at (248.0, 98.5)
- added C7: 22uf, Capacitor_THT:CP_Radial_D4.0mm_P2.00mm, F.Cu at (212.0, 118.3)
- added C8: 22uf, Capacitor_THT:CP_Radial_D4.0mm_P2.00mm, F.Cu at (253.6, 87.3)
- added C9: 22uf, Capacitor_THT:CP_Radial_D4.0mm_P2.00mm, F.Cu at (217.6, 118.3)
- added U1: 74LS00, Package_DIP:DIP-14_W7.62mm, F.Cu at (112.4, 105.0)
- added U2: 74LS161, Package_DIP:DIP-16_W7.62mm, F.Cu at (65.0, 105.0)
- added U3: 74LS161, Package_DIP:DIP-16_W7.62mm, F.Cu at (155.0, 80.0)
- added U4: 74LS161, Package_DIP:DIP-16_W7.62mm, F.Cu at (65.0, 80.0)
- added U5: 74LS161, Package_DIP:DIP-16_W7.62mm, F.Cu at (155.0, 105.0)
- added U6: 74LS245, Package_DIP:DIP-20_W7.62mm, F.Cu at (65.0, 130.0)
- added U7: 74LS245, Package_DIP:DIP-20_W7.62mm, F.Cu at (155.0, 130.0)
- moved C4 166.6 mm to (228.8, 114.3), turned to 0 degrees
- moved C1 148.0 mm to (253.6, 92.9), turned to 0 degrees
- moved C2 141.4 mm to (259.2, 87.3), turned to 0 degrees
- moved C3 128.2 mm to (280.5, 65.5), turned to 0 degrees
Connections:
- net /A15 renamed /A15 (IR.OUT.OE.INV)
- net /A16 renamed /A16 (IR.OUT.SE.INV)
- net /A17 renamed /A17 (IR.INP.INV)
- net /A18 renamed /A18 (ACC.OUT.INV)
- net /A19 renamed /A19 (ACC.INP.INV)
- net /A2 renamed /A2 (IR0)
- net /A22 renamed /A22 (RST)
- net /A3 renamed /A3 (IR1)
- net /A4 renamed /A4 (IR2)
- net /A5 renamed /A5 (IR3)
- net /A6 renamed /A6 (IR4)
- net /A7 renamed /A7 (IR5)
- net /A8 renamed /A8 (IR6)
- net /A9 renamed /A9 (IR7)
- net /B39 renamed /B39 (CLK.INV)
- J1 pad 10: /A36 -> /A36 (D3)
- J1 pad 12: /A35 -> /A35 (D4)
- J1 pad 14: /A34 -> /A34 (D5)
- J1 pad 16: /A33 -> /A33 (D6)
- J1 pad 18: /A32 -> /A32 (D7)
- J1 pad 20: /A31 -> /A31 (D8)
- J1 pad 22: /A30 -> /A30 (D9)
- J1 pad 24: /A29 -> /A29 (D10)
- J1 pad 26: /A28 -> /A28 (D11)
- J1 pad 28: /A27 -> /A27 (D12)
- J1 pad 30: /A26 -> /A26 (D13)
- J1 pad 32: /A25 -> /A25 (D14)
- J1 pad 34: /A24 -> /A24 (D15)
- J1 pad 36: /A23 -> /A23 (RST.INV)
- J1 pad 4: /A39 -> /A39 (D0)
- J1 pad 6: /A38 -> /A38 (D1)
- J1 pad 8: /A37 -> /A37 (D2)
- J2 pad 11: /B6 -> /B6 (PC.OUT)
- J2 pad 3: /B2 -> /B2 (PC.CNT)
- J2 pad 38: /B22 -> /B22 (CLK)
- J2 pad 5: /B3 -> /B3 (PC.LD)
- J2 pad 7: /B4 -> /B4 (PC.COND)
- J2 pad 9: /B5 -> /B5 (PC.LDC)
Other:
- board text added: "Andromeda Program Counter Rev. 01 7 April 2024 Copyright (C) Stanley Lancaster"
- board text removed: "Andromeda <CARD_NAME> Rev. <NUMBER> <DATE> Copyright (C) Stanley Lancaster"
