File: pcb_layouts/ProgramCount/ProgramCount.kicad_sch (KiCad schematic)
At the start: 6 parts

Commit message: pcbs
Parts:
- added C1, C10, C11, C6, C7, C8, C9: 22uf, Capacitor_THT:CP_Radial_D4.0mm_P2.00mm, symbol Device:C_Polarized
- added U1: 74LS00, Package_DIP:DIP-14_W7.62mm, symbol 74xx:74LS00
- added U2, U3, U4, U5: 74LS161, Package_DIP:DIP-16_W7.62mm, symbol 74xx:74LS161
- added U6, U7: 74LS245, Package_DIP:DIP-20_W7.62mm, symbol 74xx:74LS245
- gave numbers to parts that had none: 6
Connections:
- net A23 (RST.INV): now also U2.1 (~{MR}), U3.1 (~{MR}), U4.1 (~{MR}), U5.1 (~{MR})
- net A24 (D15): now also U5.6 (D3), U7.11 (B7)
- net A25 (D14): now also U5.5 (D2), U7.12 (B6)
- net A26 (D13): now also U5.4 (D1), U7.13 (B5)
- net A27 (D12): now also U5.3 (D0), U7.14 (B4)
- net A28 (D11): now also U3.6 (D3), U7.15 (B3)
- net A29 (D10): now also U3.5 (D2), U7.16 (B2)
- net A30 (D9): now also U3.4 (D1), U7.17 (B1)
- net A31 (D8): now also U3.3 (D0), U7.18 (B0)
- net A32 (D7): now also U4.6 (D3), U6.11 (B7)
- net A33 (D6): now also U4.5 (D2), U6.12 (B6)
- net A34 (D5): now also U4.4 (D1), U6.13 (B5)
- net A35 (D4): now also U4.3 (D0), U6.14 (B4)
- net A36 (D3): now also U2.6 (D3), U6.15 (B3)
- net A37 (D2): now also U2.5 (D2), U6.16 (B2)
- net A38 (D1): now also U2.4 (D1), U6.17 (B1)
- net A39 (D0): now also U2.3 (D0), U6.18 (B0)
- net B22 (CLK): now also U2.2 (CP), U3.2 (CP), U4.2 (CP), U5.2 (CP)
- net B3 (PC.LD): now also U1.13
- net GND: now also C1.2, C10.2, C11.2, C6.2, C7.2, C8.2, C9.2, U1.7 (GND), U2.8 (GND), U3.8 (GND), U4.8 (GND), U5.8 (GND), U6.10 (GND), U7.10 (GND)
- net VCC: now also C1.1, C10.1, C11.1, C6.1, C7.1, C8.1, C9.1, U1.12, U1.14 (VCC), U2.16 (VCC), U3.16 (VCC), U4.16 (VCC), U5.16 (VCC), U6.1 (A->B), U6.20 (VCC), U7.1 (A->B), U7.20 (VCC)
- net B2 (PC.INC) renamed B2 (PC.CNT)
- net B2 (PC.CNT): now also U2.10 (CET), U2.7 (CEP), U3.7 (CEP), U4.7 (CEP), U5.7 (CEP)
- net B4 (PC.CD) renamed B4 (PC.COND)
- net B4 (PC.COND): now also U1.4
- net B5 (PC.LCD) renamed B5 (PC.LDC)
- net B5 (PC.LDC): now also U1.5
- net B6 renamed B6 (PC.OUT)
- net B6 (PC.OUT): now also U6.19 (CE), U7.19 (CE)
- new net: U1.11, U1.9
- new net: U1.10, U1.6
- new net: U3.10 (CET), U4.15 (TC)
- new net: U3.15 (TC), U5.10 (CET)
- new net: U1.1, U1.2, U1.8
- new net: U2.15 (TC), U4.10 (CET)
- new net LD: U1.3, U2.9 (~{PE}), U3.9 (~{PE}), U4.9 (~{PE}), U5.9 (~{PE})
- new net P10: U3.12 (Q2), U7.4 (A2)
- new net P11: U3.11 (Q3), U7.5 (A3)
- new net P12: U5.14 (Q0), U7.6 (A4)
- new net P13: U5.13 (Q1), U7.7 (A5)
- new net P14: U5.12 (Q2), U7.8 (A6)
- new net P15: U5.11 (Q3), U7.9 (A7)
- new net P8: U3.14 (Q0), U7.2 (A0)
- new net P9: U3.13 (Q1), U7.3 (A1)
- new net PC0: U2.14 (Q0), U6.2 (A0)
- new net PC1: U2.13 (Q1), U6.3 (A1)
- new net PC2: U2.12 (Q2), U6.4 (A2)
- new net PC3: U2.11 (Q3), U6.5 (A3)
- new net PC4: U4.14 (Q0), U6.6 (A4)
- new net PC5: U4.13 (Q1), U6.7 (A5)
- new net PC6: U4.12 (Q2), U6.8 (A6)
- new net PC7: U4.11 (Q3), U6.9 (A7)
- no-connect marks 0 -> 1
